File: powerDistribution/symbols/powerDistributionv2.kicad_sch (KiCad schematic)
At the start: 27 parts, among them J1 Screw_Terminal_01x02, J2 Screw_Terminal_01x02, J3 Conn_01x02_Socket, J4 Conn_01x02_Socket, J5 Screw_Terminal_01x02, J6 RAPC722X, U1 LM2576-3.3, U2 LM2576HVT-5, U3 LM2678T

Commit message: brent's wifi_test_6
Parts:
- F1, F2: value 3557-10 -> ~; footprint _footprints:fz_holder_3557-10 -> 3557-10:FUSE_3557-10
- L1, L2: footprint _footprints:inductor_1A_100uH -> _footprints:1410454C_MUR
- U1: footprint _footprints:3.3V_lm2576 -> _footprints:T05A_TEX
- U2: footprint _footprints:5V_lm2576 -> _footprints:T05A_TEX
Connections:
- net CHG12V is gone; now on net +12V: J6.PIN, S1.3
- net Vout_7V_brk is gone; now on net Vout_7V: F1.2_1, J1.1 (Pin_1)
Changed lines of the file:
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@@
 	)
 	(junction
+		(at 198.12 67.31)
+		(diameter 0)
+		(color 0 0 0 0)
+	)
+	(junction
 		(at 165.1 102.87)
 		(diameter 0)
@@
 	)
 	(junction
-		(at 81.28 67.31)
-		(diameter 0)
-		(color 0 0 0 0)
-	)
-	(junction
 		(at 195.58 124.46)
 		(diameter 0)
@@
 	)
 	(junction
-		(at 198.12 67.31)
+		(at 90.17 124.46)
+		(diameter 0)
+		(color 0 0 0 0)
+	)
+	(junction
+		(at 81.28 67.31)
 		(diameter 0)
 		(color 0 0 0 0)
@@
 	(wire
 		(pts
-			(xy 83.82 124.46) (xy 95.25 124.46)
+			(xy 83.82 124.46) (xy 90.17 124.46)
 		)
 		(stroke
@@
 	(wire
 		(pts
+			(xy 81.28 67.31) (xy 83.82 67.31)
+		)
+		(stroke
+			(width 0)
+			(type default)
+		)
+	)
+	(wire
+		(pts
 			(xy 146.05 124.46) (xy 165.1 124.46)
 		)
@@
 	(wire
 		(pts
-			(xy 107.95 124.46) (xy 120.65 124.46)
+			(xy 90.17 124.46) (xy 95.25 124.46)
 		)
 		(stroke
@@
 	(wire
 		(pts
-			(xy 172.72 102.87) (xy 190.5 102.87)
+			(xy 107.95 124.46) (xy 120.65 124.46)
 		)
 		(stroke
@@
 	(wire
 		(pts
-			(xy 81.28 67.31) (xy 83.82 67.31)
+			(xy 172.72 102.87) (xy 190.5 102.87)
 		)
 		(stroke
@@
 		)
 	)
-	(label "CHG12V"
+	(label "Vin_12V"
 		(at 71.12 72.39 0)
 		(fields_autoplaced yes)
@@
 		)
 	)
-	(label "Vout_7V_brk"
+	(label "Vout_7V"
 		(at 214.63 59.69 0)
 		(fields_autoplaced yes)
@@
 	)
 	(symbol
+		(lib_id "fz_holder:3557-10")
+		(at 81.28 59.69 90)
+		(unit 1)
+		(exclude_from_sim no)
+		(in_bom yes)
+		(on_board yes)
+		(dnp no)
+		(property "Reference" "F2"
+			(at 82.804 61.214 90)
+			(effects
+				(font
+					(size 1.27 1.27)
+				)
+				(justify right)
+			)
+		)
+		(property "Value" "~"
+			(at 85.09 60.96 90)
+			(effects
+				(font
+					(size 1.27 1.27)
+				)
+				(justify right)
+			)
+		)
+		(property "Footprint" "3557-10:FUSE_3557-10"
+			(at 81.28 59.69 0)
+			(effects
+				(font
+					(size 1.27 1.27)
+				)
+				(justify bottom)
+				(hide yes)
+			)
+		)
+		(property "Datasheet" ""
+			(at 81.28 59.69 0)
+			(effects
+				(font
+					(size 1.27 1.27)
+				)
+				(hide yes)
+			)
+		)
+		(property "Description" ""
+			(at 81.28 59.69 0)
+			(effects
+				(font
+					(size 1.27 1.27)
+				)
+				(hide yes)
+			)
+		)
+		(property "PARTREV" "D"
+			(at 81.28 59.69 0)
+			(effects
+				(font
+					(size 1.27 1.27)
+				)
+				(justify bottom)
+				(hide yes)
+			)
+		)
+		(property "STANDARD" "Manufacturer Recommendation"
+			(at 81.28 59.69 0)
+			(effects
+				(font
+					(size 1.27 1.27)
+				)
+				(justify bottom)
+				(hide yes)
+			)
+		)
+		(property "SNAPEDA_PN" "3557-2"
+			(at 81.28 59.69 0)
+			(effects
+				(font
+					(size 1.27 1.27)
+				)
+				(justify bottom)
+				(hide yes)
+			)
+		)
+		(property "MAXIMUM_PACKAGE_HEIGHT" "7.37mm"
+			(at 81.28 59.69 0)
+			(effects
+				(font
+					(size 1.27 1.27)
+				)
+				(justify bottom)
+				(hide yes)
+			)
+		)
+		(property "MANUFACTURER" "Keystone"
+			(at 81.28 59.69 0)
+			(effects
+				(font
+					(size 1.27 1.27)
+				)
+				(justify bottom)
+				(hide yes)
+			)
+		)
+		(pin "2_1"
+		)
+		(pin "1_1"
+		)
+		(instances
+			(project ""
+				(path "/a5d888e0-d394-4a9f-8539-f136f21e533f"
+					(reference "F2")
+					(unit 1)
+				)
+			)
+		)
+	)
+	(symbol
 		(lib_id "power:PWR_FLAG")
 		(at 67.31 93.98 0)
@@
 	(symbol
 		(lib_id "fz_holder:3557-10")
-		(at 205.74 67.31 0)
+		(at 205.74 67.31 180)
 		(unit 1)
 		(exclude_from_sim no)
@@
 		(on_board yes)
 		(dnp no)
-		(fields_autoplaced yes)
 		(property "Reference" "F1"
-			(at 205.74 60.96 0)
+			(at 207.264 65.786 0)
 			(effects
 				(font
 					(size 1.27 1.27)
 				)
+				(justify right)
 			)
 		)
-		(property "Value" "3557-10"
-			(at 205.74 63.5 0)
+		(property "Value" "~"
+			(at 207.01 63.5 90)
 			(effects
 				(font
 					(size 1.27 1.27)
 				)
+				(justify right)
 			)
 		)
-		(property "Footprint" "_footprints:fz_holder_3557-10"
+		(property "Footprint" "3557-10:FUSE_3557-10"
 			(at 205.74 67.31 0)
 			(effects
@@
 		)
 		(instances
-			(project ""
+			(project "powerDistribution"
 				(path "/a5d888e0-d394-4a9f-8539-f136f21e533f"
 					(reference "F1")
@@
 			)
 		)
-		(property "Footprint" "_footprints:inductor_1A_100uH"
+		(property "Footprint" "_footprints:1410454C_MUR"
 			(at 132.08 116.84 0)
 			(effects
@@
 			)
 		)
-		(property "Footprint" "_footprints:5V_lm2576"
+		(property "Footprint" "_footprints:T05A_TEX"
 			(at 195.58 120.65 0)
 			(effects
@@
 		(on_board yes)
 		(dnp no)
+		(fields_autoplaced yes)
 		(property "Reference" "#PWR01"
 			(at 76.2 71.12 0)
@@
 	)
 	(symbol
-		(lib_id "fz_holder:3557-10")
-		(at 81.28 59.69 90)
-		(unit 1)
-		(exclude_from_sim no)
-		(in_bom yes)
-		(on_board yes)
-		(dnp no)
-		(fields_autoplaced yes)
-		(property "Reference" "F2"
-			(at 85.09 58.4199 90)
-			(effects
-				(font
-					(size 1.27 1.27)
-				)
-				(justify right)
-			)
-		)
-		(property "Value" "3557-10"
-			(at 85.09 60.9599 90)
-			(effects
-				(font
-					(size 1.27 1.27)
-				)
-				(justify right)
-			)
-		)
-		(property "Footprint" "_footprints:fz_holder_3557-10"
-			(at 81.28 59.69 0)
-			(effects
-				(font
-					(size 1.27 1.27)
-				)
-				(justify bottom)
-				(hide yes)
-			)
-		)
-		(property "Datasheet" ""
-			(at 81.28 59.69 0)
-			(effects
-				(font
-					(size 1.27 1.27)
-				)
-				(hide yes)
-			)
-		)
-		(property "Description" ""
-			(at 81.28 59.69 0)
-			(effects
-				(font
-					(size 1.27 1.27)
-				)
-				(hide yes)
-			)
-		)
-		(property "PARTREV" "D"
-			(at 81.28 59.69 0)
-			(effects
-				(font
-					(size 1.27 1.27)
-				)
-				(justify bottom)
-				(hide yes)
-			)
-		)
-		(property "STANDARD" "Manufacturer Recommendation"
-			(at 81.28 59.69 0)
-			(effects
-				(font
-					(size 1.27 1.27)
-				)
-				(justify bottom)
-				(hide yes)
-			)
-		)
-		(property "SNAPEDA_PN" "3557-2"
-			(at 81.28 59.69 0)
-			(effects
-				(font
-					(size 1.27 1.27)
-				)
-				(justify bottom)
-				(hide yes)
-			)
-		)
-		(property "MAXIMUM_PACKAGE_HEIGHT" "7.37mm"
-			(at 81.28 59.69 0)
-			(effects
-				(font
-					(size 1.27 1.27)
-				)
-				(justify bottom)
-				(hide yes)
-			)
-		)
-		(property "MANUFACTURER" "Keystone"
-			(at 81.28 59.69 0)
-			(effects
-				(font
-					(size 1.27 1.27)
-				)
-				(justify bottom)
-				(hide yes)
-			)
-		)
-		(pin "1_1"
-		)
-		(pin "2_1"
-		)
-		(instances
-			(project ""
-				(path "/a5d888e0-d394-4a9f-8539-f136f21e533f"
-					(reference "F2")
-					(unit 1)
-				)
-			)
-		)
-	)
-	(symbol
 		(lib_id "Device:L")
 		(at 218.44 116.84 90)
@@
 			)
 		)
-		(property "Footprint" "_footprints:inductor_1A_100uH"
+		(property "Footprint" "_footprints:1410454C_MUR"
 			(at 218.44 116.84 0)
 			(effects
@@
 			)
 		)
-		(property "Footprint" "_footprints:3.3V_lm2576"
+		(property "Footprint" "_footprints:T05A_TEX"
 			(at 107.95 120.65 0)
 			(effects
@@
 					(unit 1)
 				)
+			)
+		)
+	)
+	(symbol
+		(lib_id "power:PWR_FLAG")
+		(at 90.17 124.46 0)
+		(unit 1)
+		(exclude_from_sim no)
+		(in_bom yes)
+		(on_board yes)
+		(dnp no)
+		(fields_autoplaced yes)
+		(property "Reference" "#FLG01"
+			(at 90.17 122.555 0)
+			(effects
+				(font
+					(size 1.27 1.27)
+				)
+				(hide yes)
+			)
+		)
+		(property "Value" "PWR_FLAG"
+			(at 90.17 119.38 0)
+			(effects
+				(font
+					(size 1.27 1.27)
+				)
+			)
+		)
+		(property "Footprint" ""
+			(at 90.17 124.46 0)
+			(effects
+				(font
+					(size 1.27 1.27)
+				)
+				(hide yes)
+			)
+		)
+		(property "Datasheet" "~"
+			(at 90.17 124.46 0)
+			(effects
+				(font
+					(size 1.27 1.27)
+				)
+				(hide yes)
+			)
+		)
+		(property "Description" "Special symbol for telling ERC where power comes from"
+			(at 90.17 124.46 0)
+			(effects
+				(font
+					(size 1.27 1.27)
+				)
+				(hide yes)
+			)
+		)
+		(pin "1"
+		)
+		(instances
+			(project ""
+				(path "/a5d888e0-d394-4a9f-8539-f136f21e533f"
+					(reference "#FLG01")
+					(unit 1)
+				)
