File: pcbv2.0/pcbv2.0.kicad_sch (KiCad schematic)
At the start: 15 parts, among them J1 Screw_Terminal_01x02, J3 Screw_Terminal_01x02, U2 ESP32-DevKitC, U3 LM2576HVS-3.3, U4 LM2576HVS-5

Commit message: sync
Parts:
- removed S1: 471002268143, WE-RSTV:switch_471002268143_actual, symbol WE-RSTV:471002268143
- added SW1: S101031MS02Q, S101031MS02Q:SW2_S101031MS02Q_CNK, symbol S101031MS02Q_SPST:S101031MS02Q
- L1: value 100uH -> 1245_7447715101 (100uH)
- renumbered J3 to J2
Connections:
- net at CP4.1, L1.2, U4.4 (FB): now also SW1.1
Changed lines of the file:
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@@
 	(wire
 		(pts
-			(xy 107.95 41.91) (xy 113.03 41.91)
+			(xy 107.95 41.91) (xy 115.57 41.91)
 		)
 		(stroke
@@
 			(width 0)
 			(type default)
+		)
+	)
+	(symbol
+		(lib_id "S101031MS02Q_SPST:S101031MS02Q")
+		(at 115.57 41.91 0)
+		(unit 1)
+		(exclude_from_sim no)
+		(in_bom yes)
+		(on_board yes)
+		(dnp no)
+		(fields_autoplaced yes)
+		(property "Reference" "SW1"
+			(at 123.19 35.56 0)
+			(effects
+				(font
+					(size 1.524 1.524)
+				)
+			)
+		)
+		(property "Value" "S101031MS02Q"
+			(at 123.19 38.1 0)
+			(effects
+				(font
+					(size 1.524 1.524)
+				)
+			)
+		)
+		(property "Footprint" "S101031MS02Q:SW2_S101031MS02Q_CNK"
+			(at 115.57 41.91 0)
+			(effects
+				(font
+					(size 1.27 1.27)
+					(italic yes)
+				)
+				(hide yes)
+			)
+		)
+		(property "Datasheet" "S101031MS02Q"
+			(at 115.57 41.91 0)
+			(effects
+				(font
+					(size 1.27 1.27)
+					(italic yes)
+				)
+				(hide yes)
+			)
+		)
+		(property "Description" ""
+			(at 115.57 41.91 0)
+			(effects
+				(font
+					(size 1.27 1.27)
+				)
+				(hide yes)
+			)
+		)
+		(pin "2"
+		)
+		(pin "1"
+		)
+		(instances
+			(project ""
+				(path "/0203021d-7c2b-4845-bf22-22fcccedbbe3"
+					(reference "SW1")
+					(unit 1)
+				)
+			)
 		)
 	)
@@
 		(on_board yes)
 		(dnp no)
-		(property "Reference" "J3"
+		(property "Reference" "J2"
 			(at 140.97 62.23 0)
 			(effects
@@
 			(project "pcbv2.0"
 				(path "/0203021d-7c2b-4845-bf22-22fcccedbbe3"
-					(reference "J3")
+					(reference "J2")
 					(unit 1)
 				)
@@
 			)
 		)
-		(property "Value" "100uH"
-			(at 98.552 39.37 0)
+		(property "Value" "1245_7447715101 (100uH)"
+			(at 105.156 39.624 0)
 			(effects
 				(font
@@
 	)
 	(symbol
-		(lib_id "WE-RSTV:471002268143")
-		(at 118.11 41.91 0)
-		(unit 1)
-		(exclude_from_sim no)
-		(in_bom yes)
-		(on_board yes)
-		(dnp no)
-		(fields_autoplaced yes)
-		(property "Reference" "S1"
-			(at 118.11 35.56 0)
-			(effects
-				(font
-					(size 1.27 1.27)
-				)
-			)
-		)
-		(property "Value" "471002268143"
-			(at 118.11 38.1 0)
-			(effects
-				(font
-					(size 1.27 1.27)
-				)
-			)
-		)
-		(property "Footprint" "WE-RSTV:switch_471002268143_actual"
-			(at 118.11 41.91 0)
-			(effects
-				(font
-					(size 1.27 1.27)
-				)
-				(hide yes)
-			)
-		)
-		(property "Datasheet" ""
-			(at 118.11 41.91 0)
-			(effects
-				(font
-					(size 1.27 1.27)
-				)
-				(hide yes)
-			)
-		)
-		(property "Description" ""
-			(at 118.11 41.91 0)
-			(effects
-				(font
-					(size 1.27 1.27)
-				)
-				(hide yes)
-			)
-		)
-		(property "FRAME-COLOR" "Black"
-			(at 118.11 41.91 0)
-			(effects
-				(font
-					(size 1.27 1.27)
-				)
-				(justify bottom)
-				(hide yes)
-			)
-		)
-		(property "VALUE" "471002268143"
-			(at 118.11 41.91 0)
-			(effects
-				(font
-					(size 1.27 1.27)
-				)
-				(justify bottom)
-				(hide yes)
-			)
-		)
-		(property "QTY" "100"
-			(at 118.11 41.91 0)
-			(effects
-				(font
-					(size 1.27 1.27)
-				)
-				(justify bottom)
-				(hide yes)
-			)
-		)
-		(property "ACTUATOR-COLOR" "Black"
-			(at 118.11 41.91 0)
-			(effects
-				(font
-					(size 1.27 1.27)
-				)
-				(justify bottom)
-				(hide yes)
-			)
-		)
-		(property "DATASHEET-URL" "https://www.we-online.com/redexpert/spec/471002268143?ae"
-			(at 118.11 41.91 0)
-			(effects
-				(font
-					(size 1.27 1.27)
-				)
-				(justify bottom)
-				(hide yes)
-			)
-		)
-		(property "PART-NUMBER" "471002268143"
-			(at 118.11 41.91 0)
-			(effects
-				(font
-					(size 1.27 1.27)
-				)
-				(justify bottom)
-				(hide yes)
-			)
-		)
-		(pin "1"
-		)
-		(pin "2"
-		)
-		(instances
-			(project ""
-				(path "/0203021d-7c2b-4845-bf22-22fcccedbbe3"
-					(reference "S1")
-					(unit 1)
-				)
-			)
-		)
-	)
-	(symbol
 		(lib_id "PCM_Espressif:ESP32-DevKitC")
 		(at 67.31 152.4 0)
@@
 		(dnp no)
 		(property "Reference" "L2"
-			(at 97.536 66.04 0)
+			(at 97.536 64.262 0)
 			(effects
 				(font
@@
 		)
 		(property "Value" "1245_7447715101 (100uH)"
-			(at 105.664 70.612 0)
-			(effects
-				(font
+			(at 105.41 65.786 0)
+			(effects
+				(font
